Commit message: support cobotta robot

File: assembly_urdf_description/urdf/assembly_urdf.xacro (robot description, xacro)
@@ -23,11 +23,17 @@
     </ode>
   </physics>
-  <link name="world">
+  <!-- Connect J6(EoE of Cobotta) to the base link of gripper-->
+  <joint name="joint_gripper_base" type="fixed">
+		<parent link="J6"/>
+		<child link="gripper_base"/>
+		<origin rpy="0.000000 0.000000 0.000000" xyz="0.000000 0.000000 0.0000000"/>
+	</joint>
+  <!-- <link name="world">
   </link>
   <joint name="base_fixed_joint" type="fixed">
     <parent link="world"/>
     <child link="base_link"/>
-  </joint>
-  <link name="base_link">
+  </joint> -->
+  <link name="gripper_base_link">
     <xacro:inertia_macro radius="0.0702" height="0.1749" mass="${0.2458664564570096*hand_stiffness}">
       <origin rpy="0 0 0" xyz="0.007413303848346014 0.06187243424866449 0.052543473427993696"/>
@@ -318,5 +324,5 @@
   <joint name="r_base_hand_r" type="revolute">
     <origin rpy="0 0 0" xyz="0.014852 0.047596 0.080135"/>
-    <parent link="base_link"/>
+    <parent link="gripper_base_link"/>
     <child link="r_pinion_1"/>
     <axis xyz="0.0 0.0 1.0"/>
@@ -328,5 +334,5 @@
   <joint name="l_base_hand_r" type="revolute">
     <origin rpy="0 0 0" xyz="0.014952 0.076096 0.080135"/>
-    <parent link="base_link"/>
+    <parent link="gripper_base_link"/>
     <child link="l_pinion_1"/>
     <axis xyz="0.0 0.0 1.0"/>
@@ -337,5 +343,5 @@
   <joint name="l_base_hand_s" type="prismatic">
     <origin rpy="0 0 0" xyz="-0.095795 0.076986 0.041735"/>
-    <parent link="base_link"/>
+    <parent link="gripper_base_link"/>
     <child link="l_hand_1"/>
     <axis xyz="0.999994 -0.00352 -0.0"/>
@@ -398,5 +404,5 @@
   <joint name="r_base_hand_s" type="prismatic">
     <origin rpy="0 0 0" xyz="-0.050899 0.047328 0.041735"/>
-    <parent link="base_link"/>
+    <parent link="gripper_base_link"/>
     <child link="r_hand_1"/>
     <axis xyz="0.999994 -0.00352 -0.0"/>

Commit message: adjust relative position

File: assembly_urdf_description/urdf/assembly_urdf.xacro (robot description, xacro)
@@ -26,6 +26,6 @@
   <joint name="joint_gripper_base" type="fixed">
 		<parent link="J6"/>
-		<child link="gripper_base"/>
-		<origin rpy="0.000000 0.000000 0.000000" xyz="0.000000 0.000000 0.0000000"/>
+		<child link="gripper_base_link"/>
+		<origin rpy="0.000000 1.5708 -1.5708" xyz="-0.060000 0.060000 0.0650000"/>
 	</joint>
   <!-- <link name="world">
