Commit message: refactor name

File: gripper_ntlab_description/urdf/gripper_ntlab.xacro (robot description, xacro)
@@ -7,7 +7,7 @@
   <!--regarding there are some objects that has no inertia value-->
   <xacro:property name="hand_stiffness" value="10" />
-  <xacro:include filename="$(find assembly_urdf_description)/urdf/materials.xacro" />
-  <xacro:include filename="$(find assembly_urdf_description)/urdf/assembly_urdf.trans" />
-  <xacro:include filename="$(find assembly_urdf_description)/urdf/assembly_urdf.gazebo" />
+  <xacro:include filename="$(find gripper_ntlab_description)/urdf/materials.xacro" />
+  <xacro:include filename="$(find gripper_ntlab_description)/urdf/gripper_ntlab.trans" />
+  <xacro:include filename="$(find gripper_ntlab_description)/urdf/gripper_ntlab.gazebo" />
   <xacro:macro name="inertia_macro" params="radius height mass *origin">
     <inertial>
@@ -47,5 +47,5 @@
       <origin rpy="0 0 0" xyz="0 0 0"/>
       <geometry>
-        <mesh filename="package://assembly_urdf_description/meshes/base_link.stl" scale="0.001 0.001 0.001"/>
+        <mesh filename="package://gripper_ntlab_description/meshes/base_link.stl" scale="0.001 0.001 0.001"/>
       </geometry>
       <material name="silver_default"/>
@@ -54,5 +54,5 @@
       <origin rpy="0 0 0" xyz="0 0 0"/>
       <geometry>
-        <mesh filename="package://assembly_urdf_description/meshes/base_link.stl" scale="0.001 0.001 0.001"/>
+        <mesh filename="package://gripper_ntlab_description/meshes/base_link.stl" scale="0.001 0.001 0.001"/>
       </geometry>
     </collision>
@@ -65,5 +65,5 @@
       <origin rpy="0 0 0" xyz="0.0377 -0.047281 -0.081235"/>
       <geometry>
-        <mesh filename="package://assembly_urdf_description/meshes/r_rod_a_1.stl" scale="0.001 0.001 0.001"/>
+        <mesh filename="package://gripper_ntlab_description/meshes/r_rod_a_1.stl" scale="0.001 0.001 0.001"/>
       </geometry>
       <material name="silver_default"/>
@@ -72,5 +72,5 @@
       <origin rpy="0 0 0" xyz="0.0377 -0.047281 -0.081235"/>
       <geometry>
-        <mesh filename="package://assembly_urdf_description/meshes/r_rod_a_1.stl" scale="0.001 0.001 0.001"/>
+        <mesh filename="package://gripper_ntlab_description/meshes/r_rod_a_1.stl" scale="0.001 0.001 0.001"/>
       </geometry>
     </collision>
@@ -85,5 +85,5 @@
       <origin rpy="0 0 0" xyz="0.111195 -0.015682 -0.096135"/>
       <geometry>
-        <mesh filename="package://assembly_urdf_description/meshes/r_finger_1.stl" scale="0.001 0.001 0.001"/>
+        <mesh filename="package://gripper_ntlab_description/meshes/r_finger_1.stl" scale="0.001 0.001 0.001"/>
       </geometry>
       <material name="silver_default"/>
@@ -92,5 +92,5 @@
       <origin rpy="0 0 0" xyz="0.111195 -0.015682 -0.096135"/>
       <geometry>
-        <mesh filename="package://assembly_urdf_description/meshes/r_finger_1.stl" scale="0.001 0.001 0.001"/>
+        <mesh filename="package://gripper_ntlab_description/meshes/r_finger_1.stl" scale="0.001 0.001 0.001"/>
       </geometry>
     </collision>
@@ -105,5 +105,5 @@
       <origin rpy="0 0 0" xyz="0.172173 -0.021897 -0.092985"/>
       <geometry>
-        <mesh filename="package://assembly_urdf_description/meshes/r_roll_1.stl" scale="0.001 0.001 0.001"/>
+        <mesh filename="package://gripper_ntlab_description/meshes/r_roll_1.stl" scale="0.001 0.001 0.001"/>
       </geometry>
       <material name="silver_default"/>
@@ -112,5 +112,5 @@
       <origin rpy="0 0 0" xyz="0.172173 -0.021897 -0.092985"/>
       <geometry>
-        <mesh filename="package://assembly_urdf_description/meshes/r_roll_1.stl" scale="0.001 0.001 0.001"/>
+        <mesh filename="package://gripper_ntlab_description/meshes/r_roll_1.stl" scale="0.001 0.001 0.001"/>
       </geometry>
     </collision>
@@ -125,5 +125,5 @@
       <origin rpy="0 0 0" xyz="-0.014852 -0.047596 -0.080135"/>
       <geometry>
-        <mesh filename="package://assembly_urdf_description/meshes/r_pinion_1.stl" scale="0.001 0.001 0.001"/>
+        <mesh filename="package://gripper_ntlab_description/meshes/r_pinion_1.stl" scale="0.001 0.001 0.001"/>
       </geometry>
       <material name="silver_default"/>
@@ -132,5 +132,5 @@
       <origin rpy="0 0 0" xyz="-0.014852 -0.047596 -0.080135"/>
       <geometry>
-        <mesh filename="package://assembly_urdf_description/meshes/r_pinion_1.stl" scale="0.001 0.001 0.001"/>
+        <mesh filename="package://gripper_ntlab_description/meshes/r_pinion_1.stl" scale="0.001 0.001 0.001"/>
       </geometry>
     </collision>
@@ -145,5 +145,5 @@
       <origin rpy="0 0 0" xyz="-0.014952 -0.076096 -0.080135"/>
       <geometry>
-        <mesh filename="package://assembly_urdf_description/meshes/l_pinion_1.stl" scale="0.001 0.001 0.001"/>
+        <mesh filename="package://gripper_ntlab_description/meshes/l_pinion_1.stl" scale="0.001 0.001 0.001"/>
       </geometry>
       <material name="silver_default"/>
@@ -152,5 +152,5 @@
       <origin rpy="0 0 0" xyz="-0.014952 -0.076096 -0.080135"/>
       <geometry>
-        <mesh filename="package://assembly_urdf_description/meshes/l_pinion_1.stl" scale="0.001 0.001 0.001"/>
+        <mesh filename="package://gripper_ntlab_description/meshes/l_pinion_1.stl" scale="0.001 0.001 0.001"/>
       </geometry>
     </collision>
@@ -165,5 +165,5 @@
       <origin rpy="0 0 0" xyz="0.095795 -0.076986 -0.041735"/>
       <geometry>
-        <mesh filename="package://assembly_urdf_description/meshes/l_hand_1.stl" scale="0.001 0.001 0.001"/>
+        <mesh filename="package://gripper_ntlab_description/meshes/l_hand_1.stl" scale="0.001 0.001 0.001"/>
       </geometry>
       <material name="silver_default"/>
@@ -172,5 +172,5 @@
       <origin rpy="0 0 0" xyz="0.095795 -0.076986 -0.041735"/>
       <geometry>
-        <mesh filename="package://assembly_urdf_description/meshes/l_hand_1.stl" scale="0.001 0.001 0.001"/>
+        <mesh filename="package://gripper_ntlab_description/meshes/l_hand_1.stl" scale="0.001 0.001 0.001"/>
       </geometry>
     </collision>
@@ -183,5 +183,5 @@
       <origin rpy="0 0 0" xyz="0.036595 -0.076777 -0.08431"/>
       <geometry>
-        <mesh filename="package://assembly_urdf_description/meshes/l_rod_a_1.stl" scale="0.001 0.001 0.001"/>
+        <mesh filename="package://gripper_ntlab_description/meshes/l_rod_a_1.stl" scale="0.001 0.001 0.001"/>
       </geometry>
       <material name="abs_white"/>
@@ -190,5 +190,5 @@
       <origin rpy="0 0 0" xyz="0.036595 -0.076777 -0.08431"/>
       <geometry>
-        <mesh filename="package://assembly_urdf_description/meshes/l_rod_a_1.stl" scale="0.001 0.001 0.001"/>
+        <mesh filename="package://gripper_ntlab_description/meshes/l_rod_a_1.stl" scale="0.001 0.001 0.001"/>
       </geometry>
     </collision>
@@ -201,5 +201,5 @@
       <origin rpy="0 0 0" xyz="0.029748 -0.033397 -0.101735"/>
       <geometry>
-        <mesh filename="package://assembly_urdf_description/meshes/r_rod_b_1.stl" scale="0.001 0.001 0.001"/>
+        <mesh filename="package://gripper_ntlab_description/meshes/r_rod_b_1.stl" scale="0.001 0.001 0.001"/>
       </geometry>
       <material name="silver_default"/>
@@ -208,5 +208,5 @@
       <origin rpy="0 0 0" xyz="0.029748 -0.033397 -0.101735"/>
       <geometry>
-        <mesh filename="package://assembly_urdf_description/meshes/r_rod_b_1.stl" scale="0.001 0.001 0.001"/>
+        <mesh filename="package://gripper_ntlab_description/meshes/r_rod_b_1.stl" scale="0.001 0.001 0.001"/>
       </geometry>
     </collision>
@@ -221,5 +221,5 @@
       <origin rpy="0 0 0" xyz="0.169963 -0.09995 -0.09331"/>
       <geometry>
-        <mesh filename="package://assembly_urdf_description/meshes/l_roll_1.stl" scale="0.001 0.001 0.001"/>
+        <mesh filename="package://gripper_ntlab_description/meshes/l_roll_1.stl" scale="0.001 0.001 0.001"/>
       </geometry>
       <material name="silver_default"/>
@@ -228,5 +228,5 @@
       <origin rpy="0 0 0" xyz="0.169963 -0.09995 -0.09331"/>
       <geometry>
-        <mesh filename="package://assembly_urdf_description/meshes/l_roll_1.stl" scale="0.001 0.001 0.001"/>
+        <mesh filename="package://gripper_ntlab_description/meshes/l_roll_1.stl" scale="0.001 0.001 0.001"/>
       </geometry>
     </collision>
@@ -241,5 +241,5 @@
       <origin rpy="0 0 0" xyz="0.110234 -0.10804 -0.08456"/>
       <geometry>
-        <mesh filename="package://assembly_urdf_description/meshes/l_finger_1.stl" scale="0.001 0.001 0.001"/>
+        <mesh filename="package://gripper_ntlab_description/meshes/l_finger_1.stl" scale="0.001 0.001 0.001"/>
       </geometry>
       <material name="silver_default"/>
@@ -248,5 +248,5 @@
       <origin rpy="0 0 0" xyz="0.110234 -0.10804 -0.08456"/>
       <geometry>
-        <mesh filename="package://assembly_urdf_description/meshes/l_finger_1.stl" scale="0.001 0.001 0.001"/>
+        <mesh filename="package://gripper_ntlab_description/meshes/l_finger_1.stl" scale="0.001 0.001 0.001"/>
       </geometry>
     </collision>
@@ -259,5 +259,5 @@
       <origin rpy="0 0 0" xyz="0.028547 -0.090606 -0.089835"/>
       <geometry>
-        <mesh filename="package://assembly_urdf_description/meshes/l_rod_b_1.stl" scale="0.001 0.001 0.001"/>
+        <mesh filename="package://gripper_ntlab_description/meshes/l_rod_b_1.stl" scale="0.001 0.001 0.001"/>
       </geometry>
       <material name="silver_default"/>
@@ -266,5 +266,5 @@
       <origin rpy="0 0 0" xyz="0.028547 -0.090606 -0.089835"/>
       <geometry>
-        <mesh filename="package://assembly_urdf_description/meshes/l_rod_b_1.stl" scale="0.001 0.001 0.001"/>
+        <mesh filename="package://gripper_ntlab_description/meshes/l_rod_b_1.stl" scale="0.001 0.001 0.001"/>
       </geometry>
     </collision>
@@ -279,5 +279,5 @@
       <origin rpy="0 0 0" xyz="0.050899 -0.047328 -0.041735"/>
       <geometry>
-        <mesh filename="package://assembly_urdf_description/meshes/r_hand_1.stl" scale="0.001 0.001 0.001"/>
+        <mesh filename="package://gripper_ntlab_description/meshes/r_hand_1.stl" scale="0.001 0.001 0.001"/>
       </geometry>
       <material name="silver_default"/>
@@ -286,5 +286,5 @@
       <origin rpy="0 0 0" xyz="0.050899 -0.047328 -0.041735"/>
       <geometry>
-        <mesh filename="package://assembly_urdf_description/meshes/r_hand_1.stl" scale="0.001 0.001 0.001"/>
+        <mesh filename="package://gripper_ntlab_description/meshes/r_hand_1.stl" scale="0.001 0.001 0.001"/>
       </geometry>
     </collision>

Commit message: add property to switch between self used or with arm robot

File: gripper_ntlab_description/urdf/gripper_ntlab.xacro (robot description, xacro)
@@ -2,4 +2,6 @@
 <robot name="cobotta"
   xmlns:xacro="http://www.ros.org/wiki/xacro">
+  <xacro:arg name="base_type" default="none"/>
+  <xacro:property name="base_type" value="$(arg base_type)" />
   <xacro:property name="joint_damping" value="0.001" />
   <xacro:property name="joint_friction" value="0.61" />
@@ -24,15 +26,19 @@
   </physics>
   <!-- Connect J6(EoE of Cobotta) to the base link of gripper-->
-  <joint name="joint_gripper_base" type="fixed">
-		<parent link="J6"/>
-		<child link="gripper_base_link"/>
-		<origin rpy="0.000000 1.5708 -1.5708" xyz="-0.060000 0.060000 0.0650000"/>
-	</joint>
-  <!-- <link name="world">
-  </link>
-  <joint name="base_fixed_joint" type="fixed">
-    <parent link="world"/>
-    <child link="base_link"/>
-  </joint> -->
+  <xacro:if value="${base_type == 'cobotta'}">
+    <joint name="joint_gripper_base" type="fixed">
+      <parent link="J6"/>
+      <child link="gripper_base_link"/>
+      <origin rpy="0.000000 1.5708 -1.5708" xyz="-0.060000 0.060000 0.0650000"/>
+    </joint>
+  </xacro:if>
+  <xacro:if value="${base_type == 'none'}">
+    <link name="base_link">
+    </link>
+    <joint name="base_fixed_joint" type="fixed">
+      <parent link="base_link"/>
+      <child link="gripper_base_link"/>
+    </joint>
+  </xacro:if>
   <link name="gripper_base_link">
     <xacro:inertia_macro radius="0.0702" height="0.1749" mass="${0.2458664564570096*hand_stiffness}">

Commit message: adjust height to real position

File: gripper_ntlab_description/urdf/gripper_ntlab.xacro (robot description, xacro)
@@ -30,5 +30,5 @@
       <parent link="J6"/>
       <child link="gripper_base_link"/>
-      <origin rpy="0.000000 1.5708 -1.5708" xyz="-0.060000 0.060000 0.0650000"/>
+      <origin rpy="0.000000 1.5708 -1.5708" xyz="-0.060000 0.060000 0.1350000"/>
     </joint>
   </xacro:if>
